File: src/elec/WaMaControl/pcb/WaMaControl.kicad_pcb (KiCad board)
At the start: 2 copper layers, 225 x 125 mm, 28 parts, among them J1 Conn_01x03_Female, J2 Conn_01x04_Female, J3 Conn_01x04_Female, J4 Conn_01x02_Female, J5 Conn_01x02_Female, K1 AZ850-x, K2 AZ850-x, Q1 2SA1015, Q2 2SA1015, T1 Transformer_1P_1S, T2 Transformer_1P_1S, U1 LF50_TO220, U2 logo_fairdevices, U3 ESP32-S2-WROVER

Commit message: - migration of development files from 01-02-25
Parts:
- removed C1, C2, C3, C4, C5: C, Capacitor_THT:C_Rect_L10.3mm_W7.2mm_P7.50mm_MKS4
- removed D3, D4: 1N4001, Diode_THT:D_DO-41_SOD81_P10.16mm_Horizontal
- removed F1: Fuse, Fuse:Fuseholder_Littelfuse_445_030_series_5x25mm
- removed J1: Conn_01x03_Female, TerminalBlock_Phoenix:TerminalBlock_Phoenix_MKDS-1,5-3-5.08_1x03_P5.08mm_Horizontal
- removed J2: Conn_01x04_Female, TerminalBlock_Phoenix:TerminalBlock_Phoenix_MKDS-1,5-4-5.08_1x04_P5.08mm_Horizontal
- removed J4, J5: Conn_01x02_Female, TerminalBlock_Phoenix:TerminalBlock_Phoenix_MKDS-1,5-2-5.08_1x02_P5.08mm_Horizontal
- removed Q1: 2SA1015, Package_TO_SOT_THT:TO-92_Inline
- removed T2: Transformer_1P_1S, Transformer_THT:Transformer_Breve_TEZ-22x24
- added C100: C, Capacitor_THT:C_Rect_L10.3mm_W7.2mm_P7.50mm_MKS4, F.Cu at (131.0, 44.0)
- added C101: C, Capacitor_THT:C_Rect_L10.3mm_W7.2mm_P7.50mm_MKS4, F.Cu at (139.5, 44.0)
- added C102: C, Capacitor_THT:C_Rect_L10.3mm_W7.2mm_P7.50mm_MKS4, F.Cu at (148.0, 44.0)
- added C103: C, Capacitor_THT:C_Rect_L10.3mm_W7.2mm_P7.50mm_MKS4, F.Cu at (156.5, 44.2)
- added C104: C, Capacitor_THT:C_Rect_L10.3mm_W7.2mm_P7.50mm_MKS4, F.Cu at (173.5, 45.2)
- added C105: C, Capacitor_THT:C_Rect_L10.3mm_W7.2mm_P7.50mm_MKS4, F.Cu at (183.0, 45.2)
- added D10: 1N4001, Diode_THT:D_DO-41_SOD81_P10.16mm_Horizontal, F.Cu at (176.6, 100.0)
- added D2: 1N4001, Diode_THT:D_DO-41_SOD81_P10.16mm_Horizontal, F.Cu at (165.8, 59.8)
- added D200: 1N4001, Diode_THT:D_DO-41_SOD81_P10.16mm_Horizontal, F.Cu at (50.0, 98.5)
- added D201: 1N4001, Diode_THT:D_DO-41_SOD81_P10.16mm_Horizontal, F.Cu at (50.0, 102.8)
- added D202: 1N4001, Diode_THT:D_DO-41_SOD81_P10.16mm_Horizontal, F.Cu at (50.0, 107.0)
- added D203: 1N4001, Diode_THT:D_DO-41_SOD81_P10.16mm_Horizontal, F.Cu at (54.0, 127.5)
- added D6: 1N4001, Diode_THT:D_DO-41_SOD81_P10.16mm_Horizontal, F.Cu at (165.8, 72.5)
- added D7: D_Bridge_+-AA, Diode_THT:Diode_Bridge_Round_D8.9mm, F.Cu at (109.0, 55.5)
- added D8: 1N4001, Diode_THT:D_DO-41_SOD81_P10.16mm_Horizontal, F.Cu at (176.6, 91.5)
- added D9: 1N4001, Diode_THT:D_DO-41_SOD81_P10.16mm_Horizontal, F.Cu at (176.6, 95.7)
- added F100: Fuse, Fuse:Fuseholder_Littelfuse_445_030_series_5x25mm, F.Cu at (49.2, 34.5)
- added F101: Fuse, Fuse:Fuseholder_Littelfuse_445_030_series_5x25mm, F.Cu at (49.2, 42.5)
- added F102: Fuse, Fuse:Fuseholder_Littelfuse_445_030_series_5x25mm, F.Cu at (49.2, 50.5)
- added J100: Conn_01x03_Female, TerminalBlock_WAGO:TerminalBlock_WAGO_236-403_1x03_P5.00mm_45Degree, F.Cu at (32.5, 53.5)
- added J200: Conn_01x02_Female, TerminalBlock_Phoenix:TerminalBlock_Phoenix_MKDS-1,5-2-5.08_1x02_P5.08mm_Horizontal, F.Cu at (231.4, 89.4)
- added J201: Conn_01x02_Female, TerminalBlock_Phoenix:TerminalBlock_Phoenix_MKDS-1,5-2-5.08_1x02_P5.08mm_Horizontal, F.Cu at (231.4, 101.3)
- added J202: Conn_01x02_Female, TerminalBlock_Phoenix:TerminalBlock_Phoenix_MKDS-1,5-2-5.08_1x02_P5.08mm_Horizontal, F.Cu at (231.4, 113.1)
- added J203: Conn_01x02_Female, TerminalBlock_Phoenix:TerminalBlock_Phoenix_MKDS-1,5-2-5.08_1x02_P5.08mm_Horizontal, F.Cu at (231.4, 125.0)
- added J3: Conn_01x04_Female, TerminalBlock_Phoenix:TerminalBlock_Phoenix_MKDS-1,5-4-5.08_1x04_P5.08mm_Horizontal, F.Cu at (166.6, 83.7)
- added K202: AZ850-x, Relay_THT:Relay_SPDT_Finder_40.11, F.Cu at (132.0, 109.7)
- added K203: AZ850-x, Relay_THT:Relay_SPDT_Finder_40.11, F.Cu at (132.0, 137.5)
- added K3: AZ850-x, Relay_THT:Relay_SPDT_Finder_40.11, F.Cu at (202.8, 120.2)
- added Q12: TIC126, Package_TO_SOT_THT:TO-220-3_Vertical, F.Cu at (177.9, 106.0)
- added Q13: TIC126, Package_TO_SOT_THT:TO-220-3_Vertical, F.Cu at (177.9, 112.0)
- added Q14: TIC126, Package_TO_SOT_THT:TO-220-3_Vertical, F.Cu at (146.1, 67.5)
- added Q15: BT138-600, Package_TO_SOT_THT:TO-220-3_Vertical, F.Cu at (146.1, 73.5)
- added Q2: TIC126, Package_TO_SOT_THT:TO-220-3_Vertical, F.Cu at (146.1, 61.5)
- added R10: R_Small, Resistor_SMD:R_0805_2012Metric_Pad1.20x1.40mm_HandSolder, F.Cu at (161.5, 65.0)
- added R13: R_Small, Resistor_SMD:R_0805_2012Metric_Pad1.20x1.40mm_HandSolder, F.Cu at (187.7, 79.0)
- added R14: R_Small, Resistor_SMD:R_0805_2012Metric_Pad1.20x1.40mm_HandSolder, F.Cu at (187.7, 81.9)
- added R15: R_Small, Resistor_SMD:R_0805_2012Metric_Pad1.20x1.40mm_HandSolder, F.Cu at (187.7, 84.9)
- added R16: R_Small, Resistor_SMD:R_0805_2012Metric_Pad1.20x1.40mm_HandSolder, F.Cu at (187.7, 87.8)
- added R18: R_Small, Resistor_SMD:R_0805_2012Metric_Pad1.20x1.40mm_HandSolder, F.Cu at (161.5, 70.9)
- added R2: R_Small, Resistor_SMD:R_0805_2012Metric_Pad1.20x1.40mm_HandSolder, F.Cu at (156.8, 62.0)
- added R200: R_Small, Resistor_SMD:R_0805_2012Metric_Pad1.20x1.40mm_HandSolder, F.Cu at (64.4, 97.8)
- added R201: R_Small, Resistor_SMD:R_0805_2012Metric_Pad1.20x1.40mm_HandSolder, F.Cu at (64.4, 100.8)
- added R202: R_Small, Resistor_SMD:R_0805_2012Metric_Pad1.20x1.40mm_HandSolder, F.Cu at (64.4, 103.8)
- added R203: R_Small, Resistor_SMD:R_0805_2012Metric_Pad1.20x1.40mm_HandSolder, F.Cu at (64.4, 106.7)
- added R3: R_Small, Resistor_SMD:R_0805_2012Metric_Pad1.20x1.40mm_HandSolder, F.Cu at (156.8, 65.0)
- added R300: R_Small, Resistor_SMD:R_0805_2012Metric_Pad1.20x1.40mm_HandSolder, F.Cu at (244.4, 84.7)
- added R301: R_Small, Resistor_SMD:R_0805_2012Metric_Pad1.20x1.40mm_HandSolder, F.Cu at (244.4, 87.6)
- added R302: R_Small, Resistor_SMD:R_0805_2012Metric_Pad1.20x1.40mm_HandSolder, F.Cu at (244.4, 90.6)
- added R4: R_Small, Resistor_SMD:R_0805_2012Metric_Pad1.20x1.40mm_HandSolder, F.Cu at (156.8, 68.0)
- added R5: R_Small, Resistor_SMD:R_0805_2012Metric_Pad1.20x1.40mm_HandSolder, F.Cu at (156.8, 70.9)
- added R7: R_Small, Resistor_SMD:R_0805_2012Metric_Pad1.20x1.40mm_HandSolder, F.Cu at (156.8, 73.8)
- added U1: LF50_TO220, Package_TO_SOT_THT:TO-220-3_Vertical, F.Cu at (145.7, 94.9)
- K1, K2: value AZ850-x -> Relay_SPDT; footprint Relay_THT:Relay_DPDT_FRT5 -> Relay_THT:Relay_SPDT_Finder_40.11
- Q2: value 2SA1015 -> TIC126; footprint Package_TO_SOT_THT:TO-92_Inline -> Package_TO_SOT_THT:TO-220-3_Vertical
- moved H1 86.6 mm to (244.0, 31.5)
- moved K1 67.0 mm to (61.5, 122.0)
- moved K2 48.0 mm to (93.0, 117.5)
- moved RV1 24.4 mm to (76.5, 58.5)
- moved D1 12.1 mm to (121.1, 47.6), turned to 180 degrees
- moved T1 11.8 mm to (85.0, 37.0)
- moved U3 9.50 mm to (213.4, 66.2)
Connections:
- net Net-(T1-SA) renamed Trafo-Sek-2
- net Net-(T1-SB) renamed Trafo-Sek-1
- D1 pad 1: Net-(D1-+) -> +12V
- D1 pad 2: GND -> Earth_Protective
- J3 pad 3: motor2 -> AC/N
- Q2 pad 1: GND -> Net-(Q14-A)
- Q2 pad 2: Net-(D4-A) -> Net-(Q2-A)
- Q2 pad 3: hot-w-valve-on -> Net-(Q2-G)
- U1 pad 1: Net-(D1-+) -> +12V
- U1 pad 2: GND -> Earth_Protective
- U1 pad 3: +5V -> +3.3V
- U3 pad 1: GND -> Earth_Protective
- U3 pad 10: unconnected-(U3-IO07-Pad10) -> CNTL-coldh2o
- U3 pad 11: unconnected-(U3-IO08-Pad11) -> CNTR-warmh2o
- U3 pad 14: unconnected-(U3-IO11-Pad14) -> CNTL-drainpump
- U3 pad 19: unconnected-(U3-IO16-Pad19) -> CNTL-heating
- U3 pad 21: unconnected-(U3-IO18-Pad21) -> sens_temperature
- U3 pad 26: GND -> Earth_Protective
- U3 pad 42: GND -> Earth_Protective
- U3 pad 43: GND -> Earth_Protective
- U3 pad 5: unconnected-(U3-IO02-Pad5) -> freq
Routing:
- net Earth_Protective: track 0.00 -> 67.0 mm
- net Trafo-Sek-1: track 0.00 -> 31.8 mm
