File: src/elec/WaMaControl/pcb/WaMaControl.kicad_sch (KiCad schematic)
At the start: 5 parts, among them U2 logo_fairdevices

Commit message: - migration of development files from 01-02-25
Parts:
- U2: footprint Connector_Samtec_HPM_THT:Samtec_HPM-03-01-x-S_Straight_1x03_Pitch5.08mm -> (none)
Other:
- sheet heating-motor-valves renamed heating-valves
- added sheet motor (motor.kicad_sch)
Changed lines of the file:
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@@
 			)
 		)
-		(property "Footprint" "Connector_Samtec_HPM_THT:Samtec_HPM-03-01-x-S_Straight_1x03_Pitch5.08mm"
+		(property "Footprint" ""
 			(at 87.63 179.07 0)
 			(effects
@@
 			(color 0 0 0 0.0000)
 		)
-		(property "Sheetname" "heating-motor-valves"
+		(property "Sheetname" "heating-valves"
 			(at 85.09 25.9584 0)
 			(effects
@@
 				)
 			)
+		)
+	)
+	(sheet
+		(at 85.09 67.31)
+		(size 41.91 25.4)
+		(fields_autoplaced yes)
+		(stroke
+			(width 0.1524)
+			(type solid)
+		)
+		(fill
+			(color 0 0 0 0.0000)
+		)
+		(property "Sheetname" "motor"
+			(at 85.09 66.5984 0)
+			(effects
+				(font
+					(size 1.27 1.27)
+				)
+				(justify left bottom)
+			)
+		)
+		(property "Sheetfile" "motor.kicad_sch"
+			(at 85.09 93.2946 0)
+			(effects
+				(font
+					(size 1.27 1.27)
+				)
+				(justify left top)
+			)
+		)
+		(instances
+			(project "WaMaControl"
+				(path "/e63e39d7-6ac0-4ffd-8aa3-1841a4541b55"
+					(page "6")
+				)
+			)
