File: src/elec/WaMaControl/pcb/heating-motor-valves.kicad_sch (KiCad schematic)
At the start: 27 parts, among them J2 Conn_01x04_Female, J3 Conn_01x04_Female, J4 Conn_01x02_Female, J5 Conn_01x02_Female, K1 AZ850-x, K2 AZ850-x, Q1 2SA1015, Q2 2SA1015, Q3 BT138-600, Q4 Q_NMOS_GDS, Q5 TIC126, Q6 Q_NMOS_GDS, T3 Transformer_1P_1S, T4 Transformer_1P_1S, U4 MOC3041M

Commit message: - migration of development files from 01-02-25
Parts:
- removed D3: 1N4001, Diode_THT:D_DO-41_SOD81_P10.16mm_Horizontal, symbol Diode:1N4001
- removed J2, J3: Conn_01x04_Female, TerminalBlock_Phoenix:TerminalBlock_Phoenix_MKDS-1,5-4-5.08_1x04_P5.08mm_Horizontal, symbol Connector:Conn_01x04_Female
- removed K1, K2: AZ850-x, Relay_THT:Relay_DPDT_FRT5, symbol Relay:AZ850-x
- removed Q1, Q2: 2SA1015, Package_TO_SOT_THT:TO-92_Inline, symbol Transistor_BJT:2SA1015
- added D200, D202, D203: 1N4001, Diode_THT:D_DO-41_SOD81_P10.16mm_Horizontal, symbol Diode:1N4001
- added F3: Fuse_Small, symbol Device:Fuse_Small
- added J202, J203: Conn_01x02_Female, TerminalBlock_Phoenix:TerminalBlock_Phoenix_MKDS-1,5-2-5.08_1x02_P5.08mm_Horizontal, symbol Connector:Conn_01x02_Female
- added K1, K2, K4: Relay_SPDT, Relay_THT:Relay_SPDT_Finder_40.11, symbol Relay:Relay_SPDT
- added K202: AZ850-x, Relay_THT:Relay_SPDT_Finder_40.11, symbol Relay:AZ850-x
- added Q2: TIC126, Package_TO_SOT_THT:TO-220-3_Vertical, symbol Triac_Thyristor:TIC126
- added Q200, Q201, Q202, Q203, Q7: Q_NMOS_GDS, symbol Device:Q_NMOS_GDS
- added R10, R200, R201, R202, R203, R7: R_Small, Resistor_SMD:R_0805_2012Metric_Pad1.20x1.40mm_HandSolder, symbol Device:R_Small
- added T5: Transformer_1P_1S, symbol Device:Transformer_1P_1S
- R18: renamed from R1; footprint (none) -> Resistor_SMD:R_0805_2012Metric_Pad1.20x1.40mm_HandSolder
- R2, R3, R4, R5: footprint (none) -> Resistor_SMD:R_0805_2012Metric_Pad1.20x1.40mm_HandSolder
- renumbered C6 to C5, D5 to D12, D4 to D201, J4 to J200, J5 to J201, Q5 to Q14, Q3 to Q15, Q4 to Q5
Connections:
- net coldwatervalve1 is gone; now on net AC/N: J200.2 (Pin_2)
- net hotwatervalve1 is gone; now on net AC/N: J201.2 (Pin_2)
- net AC/L: now also F3.2, K1.14, K2.14
- net AC/N: now also J202.1 (Pin_1), J203.2 (Pin_2), K202.4, K202.8
- net GND: now also Q200.3 (S), Q201.3 (S), Q202.3 (S), Q203.3 (S), Q7.3 (S), R10.1, T5.3 (SA)
- net coldwatervalve2: now also K1.11
- net heatcontrol: no longer D6.1 (K), R5.1, T3.1 (AA)
- net heating1: now also Q14.1 (K), T4.4 (SB), J202.2 (Pin_2), K202.7, T5.2 (AB)
- net hotwatervalve2: now also K2.11
- net +12V: now reaches D201.1 (K)
- net +12V: now also D2.1 (K), D6.1 (K), T3.1 (AA), T4.1 (AA), D200.1 (K), D202.1 (K), D203.1 (K), K1.A1, K2.A1, K202.10, K4.A1
- net at D6.2 (A), T3.2 (AB): now also Q7.2 (D)
- net at T3.3 (SA): now also Q2.3 (G)
- net at T3.4 (SB): now also Q14.2 (A), F3.1, Q2.1 (K)
- net at T4.3 (SA): now also Q14.3 (G); no longer Q14.1 (K)
- net at D201.2 (A): now also K2.A2, Q201.2 (D)
- new net: D200.2 (A), K1.A2, Q200.2 (D)
- new net: D203.2 (A), K4.A2, Q203.2 (D)
- new net: Q201.1 (G), R201.2
- new net: Q2.2 (A), T5.1 (AA)
- new net: Q202.1 (G), R202.2
- new net: D202.2 (A), K202.1, Q202.2 (D)
- new net: Q200.1 (G), R200.2
- new net: Q203.1 (G), R203.2
- new net: Q7.1 (G), R7.2
- new net AC-Heating: K202.3
- new net AC-Motor: K4.12
- new net CNTL-coldh2o: R200.1
- new net CNTL-drainpump: R203.1
- new net CNTL-heating: R202.1
- new net CNTR-warmh2o: R201.1
- new net drainpump2: J203.1 (Pin_1), K4.11
- new net heatcontrol_n: R5.1
- new net heatcontrol_p: R7.1
- new net heatcurrentsens: R10.2, T5.4 (SB)
Other:
- note added: "Relais for cold water valve"
- note added: "Relais for drain pump"
- note added: "Relais for heating"
- note added: "Relais for hot water valve"
- note added: "Thyristor heat control"
- note added: "Triac Heat Control"
- note added: "current sensing for fault indication"
- note added: "freewheeling diode vs. over voltage at switch off"
- moved on the sheet: C5, D12, D2, D201, F2, J200, J201, Q14, Q15, Q5, Q6, R18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
