File: src/elec/WaMaControl/pcb/powersupply.kicad_sch (KiCad schematic)
At the start: 13 parts, among them J1 Conn_01x03_Female, T1 Transformer_1P_1S, T2 Transformer_1P_1S, U1 LF50_TO220

Commit message: - migration of development files from 01-02-25
Parts:
- removed C5: C, Capacitor_THT:C_Rect_L10.3mm_W7.2mm_P7.50mm_MKS4, symbol Device:C
- removed D7: D_Bridge_+-AA, Diode_THT:Diode_Bridge_Vishay_KBPC6, symbol Device:D_Bridge_+-AA
- removed T2: Transformer_1P_1S, Transformer_THT:Transformer_Breve_TEZ-22x24, symbol Device:Transformer_1P_1S
- added C104, C105: C, Capacitor_THT:C_Rect_L10.3mm_W7.2mm_P7.50mm_MKS4, symbol Device:C
- added F101, F102: Fuse, Fuse:Fuseholder_Littelfuse_445_030_series_5x25mm, symbol Device:Fuse
- J100: renamed from J1; footprint TerminalBlock_Phoenix:TerminalBlock_Phoenix_MKDS-1,5-3-5.08_1x03_P5.08mm_Horizontal -> TerminalBlock_WAGO:TerminalBlock_WAGO_236-403_1x03_P5.00mm_45Degree
- renumbered C1 to C100, C2 to C101, C3 to C102, C4 to C103, F1 to F100
Connections:
- net +5V is gone; now on net +3V3: U1.3 (VO)
- net +3V3: now also C104.1, C105.1
- net +12V: now reaches C100.1, C101.1, C102.1, C103.1, D1.1 (+), U1.1 (VI)
- net at F100.1, J100.3 (Pin_3): now also F101.1, F102.1
- net Trafo-Sek-2: now reaches D1.4, T1.3 (SA)
- net GND renamed Earth_Protective
- net Earth_Protective: now also C104.2, C105.2
- net freq renamed Trafo-Sek-1
- new net AC-Heating: F101.2
- new net AC-Motor: F102.2
Other:
- note added: "Electronics"
- note added: "Heating"
- note added: "Motor"
- moved on the sheet: C100, C101, C102, C103, D1, F100, J100, RV1, T1
