File: src/elec/WaMaControl/pcb/sensors.kicad_sch (KiCad schematic)
At the start: 0 parts

Commit message: - migration of development files from 01-02-25
Parts:
- added D7: D_Bridge_+-AA, Diode_THT:Diode_Bridge_Round_D8.9mm, symbol Device:D_Bridge_+-AA
- added J8: Conn_01x02_Socket, symbol Connector:Conn_01x02_Socket
- added R300, R301, R302: R_Small, Resistor_SMD:R_0805_2012Metric_Pad1.20x1.40mm_HandSolder, symbol Device:R_Small
Connections:
- new net: D7.1 (+), R300.1
- new net +3V3: R302.1
- new net GND: D7.2 (-), J8.1 (Pin_1), R301.2
- new net Trafo-Sek-1: D7.3, D7.4
- new net freq: R300.2, R301.1
- new net sens_temperature: J8.2 (Pin_2), R302.2
Other:
- note added: "Heat sensor vat"
- note added: "Power Frequency sensing"
